File: boards/base/base/_autosave-base.kicad_sch (KiCad schematic)
At the start: 25 parts, among them J1 Conn_01x04_Female, J2 Conn_01x06_Female, J3 Conn_01x06_Female, J4 Screw_Terminal_01x02, J5 Conn_01x03_Female, J6 Conn_01x02_Male, J7 Conn_01x02_Female, J8 Conn_01x03_Female, Q1 BC547, SW1 SW_Push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

Commit message: Changed routing
Parts:
- gave numbers to parts that had none: 1
Changed lines of the file:
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@@
   (symbol (lib_id "Device:R") (at 154.94 115.57 180) (unit 1)
     (in_bom yes) (on_board yes)
-    (property "Reference" "R?" (id 0) (at 152.4 115.57 90))
+    (property "Reference" "R1" (id 0) (at 152.4 115.57 90))
     (property "Value" "10k" (id 1) (at 157.48 115.57 90))
     (property "Footprint" "Resistor_THT:R_Axial_DIN0207_L6.3mm_D2.5mm_P5.08mm_Vertical" (id 2) (at 156.718 115.57 90)
@@
   (symbol (lib_id "power:GND") (at 154.94 121.92 0) (unit 1)
     (in_bom yes) (on_board yes) (fields_autoplaced)
-    (property "Reference" "#PWR?" (id 0) (at 154.94 128.27 0)
+    (property "Reference" "#PWR0107" (id 0) (at 154.94 128.27 0)
       (effects (font (size 1.27 1.27)) hide)
     )
@@
     )
     (path "/da3ebd0d-8163-4732-86d7-cc7a98cfc27a"
-      (reference "#PWR?") (unit 1) (value "GND") (footprint "")
+      (reference "#PWR0107") (unit 1) (value "GND") (footprint "")
     )
     (path "/73408e9c-10be-4e10-ba76-b1dd1086b0ce"
@@
       (reference "Q1") (unit 1) (value "BC547") (footprint "Package_TO_SOT_THT:TO-92_Inline")
     )
+    (path "/be4a9459-d6a5-4324-9fc6-fb68e81084ef"
+      (reference "R1") (unit 1) (value "10k") (footprint "Resistor_THT:R_Axial_DIN0207_L6.3mm_D2.5mm_P5.08mm_Vertical")
+    )
     (path "/7dec50cc-e90b-41bb-ace3-9f4696613882"
       (reference "R4") (unit 1) (value "10k") (footprint "Resistor_THT:R_Axial_DIN0207_L6.3mm_D2.5mm_P5.08mm_Vertical")
@@
       (reference "R8") (unit 1) (value "100") (footprint "Resistor_THT:R_Axial_DIN0207_L6.3mm_D2.5mm_P5.08mm_Vertical")
     )
-    (path "/be4a9459-d6a5-4324-9fc6-fb68e81084ef"
-      (reference "R?") (unit 1) (value "10k") (footprint "Resistor_THT:R_Axial_DIN0207_L6.3mm_D2.5mm_P5.08mm_Vertical")
-    )
     (path "/432b8744-344b-4b83-b016-4a2f511d6c04"
